Commit message: Changed radius wheels and added color

File: my_robot/urdf/my_robot.xacro (robot description, xacro)
@@ -1,4 +1,16 @@
 <robot name="my_robot" xmlns:xacro="http://www.ros.org/wiki/xacro">
 <xacro:include filename="$(find my_robot)/urdf/my_robot.gazebo" />
+  <material name="blue">
+    <color rgba= "0 0 1 1"/>
+  </material>
+  <material name="grey">
+    <color rgba="0.75 0.75 0.75 1"/>
+  </material>
+  <material name="red">
+    <color rgba="0.9 0.0 0.0 1"/>
+  </material>
+  <material name="green">
+    <color rgba="0.0 0.9 0.0 1"/>
+  </material>
   <link name="robot_footprint"></link>
   <joint name="robot_footprint_joint" type="fixed">
@@ -21,5 +33,5 @@
       <origin xyz="0 0 0" rpy=" 0 0 0"/>
       <geometry>
-        <box size=".4 .2 .1"/>
+        <box size=".42 .21 .11"/>
       </geometry>
     </collision>
@@ -27,34 +39,37 @@
       <origin xyz="0 0 0" rpy=" 0 0 0"/>
       <geometry>
-        <box size=".4 .2 .1"/>
-      </geometry>
+        <box size=".42 .21 .11"/>
+      </geometry>
+	  <material name= "red"/>
     </visual>
     <collision name='back_caster_collision'>
-      <origin xyz="-0.15 0 -0.05" rpy=" 0 0 0"/>
-      <geometry>
-        <sphere radius="0.0499"/>
+      <origin xyz="-0.15 0 -0.06" rpy=" 0 0 0"/>
+      <geometry>
+        <sphere radius="0.06"/>
       </geometry>
     </collision>
     <visual name='back_caster_visual'>
-      <origin xyz="-0.15 0 -0.05" rpy=" 0 0 0"/>
-      <geometry>
-        <sphere radius="0.05"/>
-      </geometry>
+      <origin xyz="-0.15 0 -0.06" rpy=" 0 0 0"/>
+      <geometry>
+        <sphere radius="0.06"/>
+      </geometry>
+	  <material name= "blue"/>
     </visual>
     <collision name='front_caster_collision'>
-      <origin xyz="0.15 0 -0.05" rpy=" 0 0 0"/>
-      <geometry>
-        <sphere radius="0.0499"/>
+      <origin xyz="0.15 0 -0.06" rpy=" 0 0 0"/>
+      <geometry>
+        <sphere radius="0.06"/>
       </geometry>
     </collision>
     <visual name='front_caster_visual'>
-      <origin xyz="0.15 0 -0.05" rpy=" 0 0 0"/>
-      <geometry>
-        <sphere radius="0.05"/>
-      </geometry>
+      <origin xyz="0.15 0 -0.06" rpy=" 0 0 0"/>
+      <geometry>
+        <sphere radius="0.06"/>
+      </geometry>
+	  <material name= "blue"/>
     </visual>
   </link>
 <link name='left_wheel'>
-    <pose>0 0.10 0.1 0 0 0</pose>
+    <pose>0 0.10 0.12 0 0 0</pose>
     <inertial>
       <mass value="5.0"/>
@@ -69,5 +84,5 @@
       <origin xyz="0.0 0 0" rpy=" 0 1.5705 1.5707"/>
       <geometry>
-        <cylinder radius="0.1" length ="0.05"/>
+        <cylinder radius="0.12" length ="0.05"/>
       </geometry>
     </collision>
@@ -75,10 +90,11 @@
       <origin xyz="0.0 0 0" rpy=" 0 1.5705 1.5707"/>
       <geometry>
-        <cylinder radius="0.1" length ="0.05"/>
-      </geometry>
-    </visual>
+        <cylinder radius="0.12" length ="0.05"/>
+      </geometry>
+	  <material name= "blue"/>
+	</visual>
 </link>
 <link name='right_wheel'>
-    <pose>0 -0.10 0.1 0 0 0</pose>
+    <pose>0 -0.10 0.12 0 0 0</pose>
     <inertial>
       <mass value="5.0"/>
@@ -93,5 +109,5 @@
       <origin xyz="0.0 0 0" rpy=" 0 1.5705 1.5707"/>
       <geometry>
-        <cylinder radius="0.1" length ="0.05"/>
+        <cylinder radius="0.12" length ="0.05"/>
       </geometry>
     </collision>
@@ -99,6 +115,7 @@
       <origin xyz="0.0 0 0" rpy=" 0 1.5705 1.5707"/>
       <geometry>
-        <cylinder radius="0.1" length ="0.05"/>
-      </geometry>
+        <cylinder radius="0.12" length ="0.05"/>
+      </geometry>
+	  <material name= "blue"/>
     </visual>
 </link>
@@ -125,4 +142,5 @@
         <box size=".05 .05 .05"/>
       </geometry>
+	  <material name= "green"/>
     </visual>
 </link>
@@ -179,3 +197,16 @@
     <axis xyz="0 1 0" rpy="0 0 0"/>s
   </joint>
+  <!-- Color the components in Gazebo-->
+  <gazebo reference="chassis">
+    <material>Gazebo/Red</material>
+  </gazebo>
+  <gazebo reference="left_wheel">
+    <material>Gazebo/Green</material>
+  </gazebo>
+  <gazebo reference="right_wheel">
+    <material>Gazebo/Green</material>
+  </gazebo>
+  <gazebo reference="camera">
+    <material>Gazebo/Blue</material>
+  </gazebo>
 </robot>
